File: hardware/V3.4.2/emonTx V3.4.2.sch (EAGLE design)
At the start: 100 parts, among them CN1 2.1MM, IC2 7805, J3 1X2-3.5MM, J5 1X2-3.5MM, J6 1X2-3.5MM, Q1 16Mhz, U1 ATMEGA168MLF, U1_TQFP ATMEGA328P

Commit message: update board and schematic images to latest V3.4.2
Other:
- note added: "OpenEnergyMonitor.org"
- note added: "emonTx V3.4.2"
- note removed: "emonTx V3.4 OpenEnergyMonitor.org"
- note removed: "emonTx V3.4.1"
Changed lines of the file:
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@@
 <?xml version="1.0" encoding="utf-8"?>
 <!DOCTYPE eagle SYSTEM "eagle.dtd">
-<eagle version="7.6.0">
+<eagle version="8.3.1">
 <drawing>
 <settings>
 <setting alwaysvectorfont="no"/>
+<setting keepoldvectorfont="yes"/>
 <setting verticaltext="up"/>
 </settings>
@@
 <plain>
 <text x="0" y="271.78" size="1.778" layer="91">AC-AC 9V measurement</text>
-<text x="214.63" y="204.47" size="1.778" layer="91">emonTx V3.4
-OpenEnergyMonitor.org</text>
+<text x="214.63" y="204.47" size="1.778" layer="91">OpenEnergyMonitor.org</text>
 <text x="214.63" y="200.66" size="1.778" layer="91">Glyn Hudson  -  March 2015</text>
 <wire x1="-99.06" y1="393.7" x2="-25.4" y2="393.7" width="0.1524" layer="94"/>
@@
 <text x="-83.82" y="190.5" size="1.778" layer="91">Design is provided "AS IS" and "WITH ALL FAULTS. OpenEnergyMonitor DISCLAIMS ALL OTHER WARRANTIES, EXPRESS OR IMPLIED,</text>
 <text x="-83.82" y="194.31" size="1.778" layer="91">Hardware design files are licensed under the Creative Commons Attribution-ShareAlike 3.0 Unported License</text>
-<text x="-97.79" y="396.24" size="5.08" layer="91">emonTx V3.4.1</text>
+<text x="-97.79" y="396.24" size="5.08" layer="91">emonTx V3.4.2</text>
 <text x="1.27" y="360.68" size="1.778" layer="91">D19 / ADC 5 DS18B20 PWR</text>
 <text x="1.27" y="363.22" size="1.778" layer="91">D5 - one-wire data</text>
@@
 <pinref part="R13" gate="G$1" pin="2"/>
 <junction x="7.62" y="259.08"/>
-<pinref part="R13" gate="G$1" pin="2"/>
-</segment>
-</net>
+</segment>
+</net>
